File: pcb/elephant42.kicad_pcb (KiCad board)
At the start: 2 copper layers, 139.4 x 124 mm, 64 parts, among them J1 MJ-4PP-9, J2 LED, SW1 SW_PUSH, SW10 SW_PUSH, SW11 SW_PUSH, SW12 SW_PUSH, SW13 SW_PUSH, SW14 SW_PUSH, SW15 SW_PUSH, SW16 SW_PUSH, SW17 SW_PUSH, SW18 SW_PUSH, SW19 SW_PUSH, SW2 SW_PUSH, SW20 SW_PUSH, SW21 SW_PUSH, SW3 SW_PUSH, SW4 SW_PUSH, SW5 SW_PUSH, SW6 SW_PUSH, SW7 SW_PUSH, SW8 SW_PUSH, SW9 SW_PUSH, U1 ProMicro

Commit message: add LED
Parts:
- removed G***: LOGO, elephant42:icon
- removed G***: LOGO, elephant42:logo
- removed JP1, JP2, JP3, JP4, JP5, JP6, JP7, JP8: Jumper, kbd:Jumper
- added D22: D, kbd:D3_SMD_v2, B.Cu at (201.5, 41.7)
- added D23: D, kbd:D3_SMD_v2, B.Cu at (222.9, 32.2)
- added D24: D, kbd:D3_SMD_v2, B.Cu at (239.6, 27.4)
- added D25: D, kbd:D3_SMD_v2, B.Cu at (261.0, 27.4)
- added D26: D, kbd:D3_SMD_v2, B.Cu at (277.7, 48.9)
- added D27: D, kbd:D3_SMD_v2, B.Cu at (299.1, 53.6)
- added D28: D, kbd:D3_SMD_v2, B.Cu at (203.8, 56.0)
- added D29: D, kbd:D3_SMD_v2, B.Cu at (222.9, 51.3)
- added D30: D, kbd:D3_SMD_v2, B.Cu at (241.9, 41.7)
- added D31: D, kbd:D3_SMD_v2, B.Cu at (261.0, 46.5)
- added D32: D, kbd:D3_SMD_v2, B.Cu at (280.0, 63.2)
- added D33: D, kbd:D3_SMD_v2, B.Cu at (299.1, 72.7)
- added D34: D, kbd:D3_SMD_v2, B.Cu at (205.0, 71.5)
- added D35: D, kbd:D3_SMD_v2, B.Cu at (224.1, 63.2)
- added D36: D, kbd:D3_SMD_v2, B.Cu at (241.9, 60.8)
- added D37: D, kbd:D3_SMD_v2, B.Cu at (261.0, 65.5)
- added D38: D, kbd:D3_SMD_v2, B.Cu at (280.0, 82.2)
- added D39: D, kbd:D3_SMD_v2, B.Cu at (180.0, 116.7)
- added D40: D, kbd:D3_SMD_v2, B.Cu at (196.7, 103.6)
- added D41: D, kbd:D3_SMD_v2, B.Cu at (215.7, 96.5)
- added D42: D, kbd:D3_SMD_v2, B.Cu at (236.0, 94.1)
- added H10: MountingHole, kbd:HOLE, F.Cu at (147.4, 116.7)
- added H11: MountingHole, kbd:HOLE, F.Cu at (50.2, 54.8)
- added H12: MountingHole, kbd:HOLE, F.Cu at (165.1, 116.7)
- added H13: MountingHole, kbd:HOLE, F.Cu at (243.1, 27.7)
- added H14: MountingHole, kbd:HOLE, F.Cu at (107.4, 37.3)
- added H8: MountingHole, kbd:HOLE, F.Cu at (262.2, 54.8)
- added H9: MountingHole, kbd:HOLE, F.Cu at (281.2, 45.9)
- added J3: MJ-4PP-9, kbd:MJ-4PP-9_1side, F.Cu at (167.0, 84.8)
- added J4: LED, kbd:StripLED_1side, B.Cu at (172.2, 64.1)
- added L1: SK6812MINI, kbd:SK6812MINI, F.Cu at (84.0, 97.7)
- added L10: SK6812MINI, kbd:SK6812MINI, F.Cu at (97.9, 73.9)
- added L11: SK6812MINI, kbd:SK6812MINI, F.Cu at (78.8, 64.4)
- added L12: SK6812MINI, kbd:SK6812MINI, F.Cu at (78.8, 45.3)
- added L13: SK6812MINI, kbd:SK6812MINI, F.Cu at (78.8, 26.3)
- added L14: SK6812MINI, kbd:SK6812MINI, F.Cu at (59.8, 31.0)
- added L15: SK6812MINI, kbd:SK6812MINI, F.Cu at (59.8, 50.1)
- added L16: SK6812MINI, kbd:SK6812MINI, F.Cu at (59.8, 69.1)
- added L17: SK6812MINI, kbd:SK6812MINI, F.Cu at (40.7, 85.8)
- added L18: SK6812MINI, kbd:SK6812MINI, F.Cu at (40.7, 66.7)
- added L19: SK6812MINI, kbd:SK6812MINI, F.Cu at (40.7, 47.7)
- added L2: SK6812MINI, kbd:SK6812MINI, F.Cu at (103.5, 102.5)
- added L20: SK6812MINI, kbd:SK6812MINI, F.Cu at (21.7, 57.2)
- added L21: SK6812MINI, kbd:SK6812MINI, F.Cu at (21.7, 76.3)
- added L22: SK6812MINI, kbd:SK6812MINI_underglow, F.Cu at (50.6, 72.0)
- added L23: SK6812MINI, kbd:SK6812MINI_underglow, F.Cu at (51.6, 35.9)
- added L24: SK6812MINI, kbd:SK6812MINI_underglow, F.Cu at (89.0, 23.7)
- added L25: SK6812MINI, kbd:SK6812MINI_underglow, F.Cu at (137.2, 54.9)
- added L26: SK6812MINI, kbd:SK6812MINI_underglow, F.Cu at (135.4, 94.3)
- added L27: SK6812MINI, kbd:SK6812MINI_underglow, F.Cu at (97.2, 88.9)
- added L28: SK6812MINI, kbd:SK6812MINI, F.Cu at (228.2, 97.7)
- added L29: SK6812MINI, kbd:SK6812MINI, F.Cu at (208.8, 102.6)
- added L3: SK6812MINI, kbd:SK6812MINI, F.Cu at (121.0, 112.4)
- added L30: SK6812MINI, kbd:SK6812MINI, F.Cu at (191.5, 112.4)
- added L31: SK6812MINI, kbd:SK6812MINI, F.Cu at (177.1, 126.3)
- added L32: SK6812MINI, kbd:SK6812MINI, F.Cu at (195.5, 78.6)
- added L33: SK6812MINI, kbd:SK6812MINI, F.Cu at (195.5, 59.6)
- added L34: SK6812MINI, kbd:SK6812MINI, F.Cu at (195.5, 40.5)
- added L35: SK6812MINI, kbd:SK6812MINI, F.Cu at (214.6, 35.8)
- added L36: SK6812MINI, kbd:SK6812MINI, F.Cu at (214.6, 54.8)
- added L37: SK6812MINI, kbd:SK6812MINI, F.Cu at (214.6, 73.9)
- added L38: SK6812MINI, kbd:SK6812MINI, F.Cu at (233.6, 64.4)
- added L39: SK6812MINI, kbd:SK6812MINI, F.Cu at (233.6, 45.3)
- added L4: SK6812MINI, kbd:SK6812MINI, F.Cu at (135.3, 126.3)
- added L40: SK6812MINI, kbd:SK6812MINI, F.Cu at (233.6, 26.3)
- added L41: SK6812MINI, kbd:SK6812MINI, F.Cu at (252.7, 31.0)
- added L42: SK6812MINI, kbd:SK6812MINI, F.Cu at (252.7, 50.1)
- added L43: SK6812MINI, kbd:SK6812MINI, F.Cu at (252.7, 69.1)
- added L44: SK6812MINI, kbd:SK6812MINI, F.Cu at (271.7, 85.8)
- added L45: SK6812MINI, kbd:SK6812MINI, F.Cu at (271.7, 66.7)
- added L46: SK6812MINI, kbd:SK6812MINI, F.Cu at (271.7, 47.7)
- added L47: SK6812MINI, kbd:SK6812MINI, F.Cu at (290.8, 57.2)
- added L48: SK6812MINI, kbd:SK6812MINI, F.Cu at (290.8, 76.3)
- added L49: SK6812MINI, kbd:SK6812MINI_underglow, F.Cu at (261.1, 71.5)
- added L5: SK6812MINI, kbd:SK6812MINI, F.Cu at (116.9, 78.6)
- added L50: SK6812MINI, kbd:SK6812MINI_underglow, F.Cu at (261.7, 36.3)
- added L51: SK6812MINI, kbd:SK6812MINI_underglow, F.Cu at (225.6, 24.6)
- added L52: SK6812MINI, kbd:SK6812MINI_underglow, F.Cu at (174.9, 54.3)
- added L53: SK6812MINI, kbd:SK6812MINI_underglow, F.Cu at (177.7, 94.5)
- added L54: SK6812MINI, kbd:SK6812MINI_underglow, F.Cu at (215.7, 88.2)
- added L6: SK6812MINI, kbd:SK6812MINI, F.Cu at (116.9, 59.6)
- added L7: SK6812MINI, kbd:SK6812MINI, F.Cu at (116.9, 40.5)
- added L8: SK6812MINI, kbd:SK6812MINI, F.Cu at (97.9, 35.8)
- added L9: SK6812MINI, kbd:SK6812MINI, F.Cu at (97.9, 54.8)
- added OL2: OLED, kbd:OLED_1side, F.Cu at (132.7, 78.6)
- added RESET_SW2: SW_PUSH, kbd:ResetSW, F.Cu at (172.8, 90.0)
- added SW22: SW_PUSH, kbd:CherryMX_Hotswap, F.Cu at (195.5, 35.8)
- added SW23: SW_PUSH, kbd:CherryMX_Hotswap, F.Cu at (214.6, 31.0)
- added SW24: SW_PUSH, kbd:CherryMX_Hotswap, F.Cu at (233.6, 21.5)
- added SW25: SW_PUSH, kbd:CherryMX_Hotswap, F.Cu at (252.7, 26.3)
- added SW26: SW_PUSH, kbd:CherryMX_Hotswap, F.Cu at (271.7, 42.9)
- added SW27: SW_PUSH, kbd:CherryMX_Hotswap, F.Cu at (290.8, 52.5)
- added SW28: SW_PUSH, kbd:CherryMX_Hotswap, F.Cu at (195.5, 54.8)
- added SW29: SW_PUSH, kbd:CherryMX_Hotswap, F.Cu at (214.6, 50.1)
- added SW30: SW_PUSH, kbd:CherryMX_Hotswap, F.Cu at (233.6, 40.5)
- added SW31: SW_PUSH, kbd:CherryMX_Hotswap, F.Cu at (252.7, 45.3)
- added SW32: SW_PUSH, kbd:CherryMX_Hotswap, F.Cu at (271.7, 62.0)
- added SW33: SW_PUSH, kbd:CherryMX_Hotswap, F.Cu at (290.8, 71.5)
- added SW34: SW_PUSH, kbd:CherryMX_Hotswap, F.Cu at (195.5, 73.9)
- added SW35: SW_PUSH, kbd:CherryMX_Hotswap, F.Cu at (214.6, 69.1)
- added SW36: SW_PUSH, kbd:CherryMX_Hotswap, F.Cu at (233.6, 59.6)
- added SW37: SW_PUSH, kbd:CherryMX_Hotswap, F.Cu at (252.7, 64.4)
- added SW38: SW_PUSH, kbd:CherryMX_Hotswap, F.Cu at (271.7, 81.0)
- added SW39: SW_PUSH, kbd:CherryMX_Hotswap, F.Cu at (173.8, 123.0)
- added SW40: SW_PUSH, kbd:CherryMX_Hotswap, F.Cu at (189.0, 108.3)
- added SW41: SW_PUSH, kbd:CherryMX_Hotswap, F.Cu at (207.6, 98.0)
- added SW42: SW_PUSH, kbd:CherryMX_Hotswap, F.Cu at (228.2, 92.9)
- added U2: ProMicro, kbd:ProMicro_v3, F.Cu at (175.9, 62.3)
- D1, D10, D11, D12, D13, D14, D15, D16, D17, D18, D19, D2, D20, D21, D3, D4, D5, D6, D7, D8, D9: footprint kbd:D3_TH_SMD -> kbd:D3_SMD_v2; moved to B.Cu
- J1: footprint kbd:MJ-4PP-9 -> kbd:MJ-4PP-9_1side
- J2: footprint kbd:StripLED_rev -> kbd:StripLED_1side; moved to B.Cu
- OL1: footprint kbd:OLED -> kbd:OLED_1side
- U1: footprint kbd:ProMicro_v2 -> kbd:ProMicro_v3
- moved H4 138.7 mm to (31.2, 45.9)
- moved J2 122.3 mm to (139.4, 70.3)
- moved H6 116.5 mm to (205.0, 37.3)
- moved H2 101.9 mm to (200.7, 109.0)
- moved H1 99.7 mm to (111.8, 109.0)
- moved H7 98.0 mm to (205.0, 61.6)
- moved H3 55.0 mm to (107.4, 61.6)
- moved OL1 37.7 mm to (172.3, 78.5)
- moved D20 11.3 mm to (135.7, 107.6), turned to 45 degrees
- moved J1 11.1 mm to (145.4, 84.7)
- moved D18 9.41 mm to (92.7, 93.5), turned to 90 degrees
- moved D17 8.42 mm to (125.3, 73.9), turned to 90 degrees
- moved D9 8.42 mm to (68.1, 45.3), turned to 90 degrees
- moved D14 8.42 mm to (68.1, 64.4), turned to 90 degrees
- moved D2 8.42 mm to (49.1, 42.9), turned to 90 degrees
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Connections:
- net data renamed data_l
- net reset renamed reset_l
- J1 pad A: Net-(J1-PadA) -> (no net)
- J2 pad 1: GND -> VCC
- J2 pad 2: led -> Net-(J2-Pad2)
- J2 pad 3: VCC -> GND
- OL1 pad 1: Net-(JP1-Pad2) -> sda_r
- OL1 pad 2: Net-(JP2-Pad2) -> scl_r
- OL1 pad 3: Net-(JP3-Pad2) -> VCC
- OL1 pad 4: Net-(JP4-Pad2) -> GND
- U1 pad 1: led -> led_l
- U1 pad 11: Net-(U1-Pad11) -> (no net)
- U1 pad 12: Net-(U1-Pad12) -> (no net)
- U1 pad 13: Net-(U1-Pad13) -> (no net)
- U1 pad 14: Net-(U1-Pad14) -> (no net)
- U1 pad 24: Net-(U1-Pad24) -> (no net)
- U1 pad 5: sda -> sda_l
- U1 pad 6: scl -> scl_l
Routing:
- net GND: track 228.9 -> 1235.6 mm, vias 23 -> 38
- net VCC: track 250.3 -> 1219.2 mm, vias 3 -> 32
- net col8: track 0.00 -> 201.4 mm, vias 0 -> 1
- net row4: track 0.00 -> 170.1 mm, vias 0 -> 7
- net col9: track 0.00 -> 164.9 mm, vias 0 -> 1
- net col6: track 0.00 -> 153.2 mm, vias 0 -> 1
- net row5: track 0.00 -> 149.4 mm, vias 0 -> 8
- net col7: track 0.00 -> 149.0 mm, vias 0 -> 1
- net led: track 141.3 -> 0.00 mm, vias 3 -> 0
- net row7: track 0.00 -> 130.5 mm, vias 0 -> 2
- net col10: track 0.00 -> 128.6 mm, vias 0 -> 1
- net row6: track 0.00 -> 128.2 mm, vias 0 -> 5
- net col11: track 0.00 -> 127.2 mm, vias 0 -> 1
- net led_l: track 0.00 -> 120.8 mm, vias 0 -> 1
- net led_r: track 0.00 -> 105.7 mm, vias 0 -> 3
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- removed copper zone on B.Cu, net GND
- removed copper zone on F.Cu, net GND
Other:
- board size 139.4 x 124 mm -> 288.1 x 124 mm
- board text removed: "Elephant42 [Beta] designed by @illness072"

Commit message: jlcpcb
Parts:
- removed H1, H10, H11, H12, H13, H14, H2, H3, H4, H5, H6, H7, H8, H9: MountingHole, kbd:HOLE
- removed J2, J4: LED, kbd:StripLED_1side
- added L55: YS-SK6812mini-E, maou_kbd:YS-SK6812MINI-E-underglow, F.Cu at (66.2, 134.4)
- added L56: LED, kbd:StripLED_1side, F.Cu at (24.6, 160.6)
- D22, D23, D24, D25, D26, D27, D28, D29, D30, D31, D32, D33, D34, D35, D36, D37, D38, D39, D40, D41, D42: moved to F.Cu
- J3, OL1, RESET_SW2, SW22, SW23, SW24, SW25, SW26, SW27, SW28, SW29, SW30, SW31, SW32, SW33, SW34, SW35, SW36, SW37, SW38, SW39, SW40, SW41, SW42, U2: moved to B.Cu
- L1, L10, L11, L12, L13, L14, L15, L16, L17, L18, L19, L2, L20, L21, L3, L4, L5, L6, L7, L8, L9: value SK6812MINI -> YS-SK6812mini-E; footprint kbd:SK6812MINI -> maou_kbd:YS-SK6812MINI-E; moved to B.Cu
- L22, L23, L24, L25, L26, L27: value SK6812MINI -> YS-SK6812mini-E; footprint kbd:SK6812MINI_underglow -> maou_kbd:YS-SK6812MINI-E-underglow; moved to B.Cu
- L28: value SK6812MINI -> LED; footprint kbd:SK6812MINI -> kbd:StripLED_1side; moved to B.Cu
- L29, L30, L31, L32, L33, L34, L35, L36, L37, L38, L39, L40, L41, L42, L43, L44, L45, L46, L47, L48: value SK6812MINI -> YS-SK6812mini-E; footprint kbd:SK6812MINI -> maou_kbd:YS-SK6812MINI-E
- L49: value SK6812MINI -> YS-SK6812mini-E; footprint kbd:SK6812MINI_underglow -> maou_kbd:YS-SK6812MINI-E
- L50, L51, L52, L53, L54: value SK6812MINI -> YS-SK6812mini-E; footprint kbd:SK6812MINI_underglow -> maou_kbd:YS-SK6812MINI-E-underglow
- moved L41 243.8 mm to (85.3, 208.2), turned to 0 degrees
- moved D24 241.6 mm to (79.3, 208.2)
- moved D25 237.8 mm to (96.0, 198.7)
- moved SW24 234.8 mm to (85.3, 203.5), turned to 180 degrees
- moved D23 232.7 mm to (60.3, 198.7)
- moved L35 230.3 mm to (47.2, 194.0), turned to 0 degrees
- moved SW25 227.5 mm to (104.3, 198.7), turned to 180 degrees
- moved SW23 220.3 mm to (66.2, 194.0), turned to 180 degrees
- moved L40 220.3 mm to (85.3, 189.2), turned to 0 degrees
- moved D22 219.5 mm to (38.9, 189.2)
- moved D30 217.3 mm to (76.9, 183.1)
- moved L42 213.4 mm to (104.3, 203.5), turned to 0 degrees
- moved SW22 213.4 mm to (47.2, 189.2), turned to 180 degrees
- moved D31 212.0 mm to (96.0, 179.7)
- moved L47 211.7 mm to (123.4, 186.8), turned to 0 degrees
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Connections:
- L1 pad 1: Net-(L1-Pad1) -> VCC
- L1 pad 2: GND -> Net-(L1-Pad2)
- L1 pad 3: led_l -> GND
- L1 pad 4: VCC -> led_l
- L10 pad 1: Net-(L10-Pad1) -> VCC
- L10 pad 2: GND -> Net-(L10-Pad2)
- L10 pad 3: Net-(L10-Pad3) -> GND
- L10 pad 4: VCC -> Net-(L10-Pad4)
- L11 pad 1: Net-(L11-Pad1) -> VCC
- L11 pad 2: GND -> Net-(L11-Pad2)
- L11 pad 3: Net-(L10-Pad1) -> GND
- L11 pad 4: VCC -> Net-(L10-Pad2)
- L12 pad 1: Net-(L12-Pad1) -> VCC
- L12 pad 2: GND -> Net-(L12-Pad2)
- L12 pad 3: Net-(L11-Pad1) -> GND
- L12 pad 4: VCC -> Net-(L11-Pad2)
- L13 pad 1: Net-(L13-Pad1) -> VCC
- L13 pad 2: GND -> Net-(L13-Pad2)
- L13 pad 3: Net-(L12-Pad1) -> GND
- L13 pad 4: VCC -> Net-(L12-Pad2)
- L14 pad 1: Net-(L14-Pad1) -> VCC
- L14 pad 2: GND -> Net-(L14-Pad2)
- L14 pad 3: Net-(L13-Pad1) -> GND
- L14 pad 4: VCC -> Net-(L13-Pad2)
- L15 pad 1: Net-(L15-Pad1) -> VCC
- L15 pad 2: GND -> Net-(L15-Pad2)
- L15 pad 3: Net-(L14-Pad1) -> GND
- L15 pad 4: VCC -> Net-(L14-Pad2)
- L16 pad 1: Net-(L16-Pad1) -> VCC
- L16 pad 2: GND -> Net-(L16-Pad2)
- L16 pad 3: Net-(L15-Pad1) -> GND
- L16 pad 4: VCC -> Net-(L15-Pad2)
- L17 pad 1: Net-(L17-Pad1) -> VCC
- L17 pad 2: GND -> Net-(L17-Pad2)
- L17 pad 3: Net-(L16-Pad1) -> GND
- L17 pad 4: VCC -> Net-(L16-Pad2)
- L18 pad 1: Net-(L18-Pad1) -> VCC
- L18 pad 2: GND -> Net-(L18-Pad2)
- L18 pad 3: Net-(L17-Pad1) -> GND
- L18 pad 4: VCC -> Net-(L17-Pad2)
- L19 pad 1: Net-(L19-Pad1) -> VCC
- L19 pad 2: GND -> Net-(L19-Pad2)
- L19 pad 3: Net-(L18-Pad1) -> GND
- L19 pad 4: VCC -> Net-(L18-Pad2)
- L2 pad 1: Net-(L2-Pad1) -> VCC
- L2 pad 2: GND -> Net-(L2-Pad2)
- L2 pad 3: Net-(L1-Pad1) -> GND
- L2 pad 4: VCC -> Net-(L1-Pad2)
- L20 pad 1: Net-(L20-Pad1) -> VCC
- L20 pad 2: GND -> Net-(L20-Pad2)
- L20 pad 3: Net-(L19-Pad1) -> GND
- L20 pad 4: VCC -> Net-(L19-Pad2)
- L21 pad 1: Net-(L21-Pad1) -> VCC
- L21 pad 2: GND -> Net-(L21-Pad2)
- L21 pad 3: Net-(L20-Pad1) -> GND
- L21 pad 4: VCC -> Net-(L20-Pad2)
- L22 pad 1: Net-(L22-Pad1) -> VCC
- L22 pad 2: GND -> Net-(L22-Pad2)
- L22 pad 3: Net-(L21-Pad1) -> GND
- L22 pad 4: VCC -> Net-(L21-Pad2)
- L23 pad 1: Net-(L23-Pad1) -> VCC
- L23 pad 2: GND -> Net-(L23-Pad2)
- L23 pad 3: Net-(L22-Pad1) -> GND
- L23 pad 4: VCC -> Net-(L22-Pad2)
- L24 pad 1: Net-(L24-Pad1) -> VCC
- L24 pad 2: GND -> Net-(L24-Pad2)
- L24 pad 3: Net-(L23-Pad1) -> GND
- L24 pad 4: VCC -> Net-(L23-Pad2)
- L25 pad 1: Net-(L25-Pad1) -> VCC
- L25 pad 2: GND -> Net-(L25-Pad2)
- L25 pad 3: Net-(L24-Pad1) -> GND
- L25 pad 4: VCC -> Net-(L24-Pad2)
- L26 pad 1: Net-(L26-Pad1) -> VCC
- L26 pad 2: GND -> Net-(L26-Pad2)
- L26 pad 3: Net-(L25-Pad1) -> GND
- L26 pad 4: VCC -> Net-(L25-Pad2)
- L27 pad 1: Net-(J2-Pad2) -> VCC
- L27 pad 2: GND -> Net-(L27-Pad2)
- L27 pad 3: Net-(L26-Pad1) -> GND
- L27 pad 4: VCC -> Net-(L26-Pad2)
- L28 pad 1: Net-(L28-Pad1) -> VCC
- L28 pad 2: GND -> Net-(L27-Pad2)
- L28 pad 3: led_r -> GND
- L29 pad 1: Net-(L29-Pad1) -> VCC
- L29 pad 2: GND -> Net-(L29-Pad2)
- L29 pad 3: Net-(L28-Pad1) -> GND
- L29 pad 4: VCC -> led_r
- L3 pad 1: Net-(L3-Pad1) -> VCC
- L3 pad 2: GND -> Net-(L3-Pad2)
- L3 pad 3: Net-(L2-Pad1) -> GND
- L3 pad 4: VCC -> Net-(L2-Pad2)
- L30 pad 1: Net-(L30-Pad1) -> VCC
- L30 pad 2: GND -> Net-(L30-Pad2)
- L30 pad 3: Net-(L29-Pad1) -> GND
- L30 pad 4: VCC -> Net-(L29-Pad2)
- L31 pad 1: Net-(L31-Pad1) -> VCC
- L31 pad 2: GND -> Net-(L31-Pad2)
- L31 pad 3: Net-(L30-Pad1) -> GND
- L31 pad 4: VCC -> Net-(L30-Pad2)
- L32 pad 1: Net-(L32-Pad1) -> VCC
- L32 pad 2: GND -> Net-(L32-Pad2)
- L32 pad 3: Net-(L31-Pad1) -> GND
- L32 pad 4: VCC -> Net-(L31-Pad2)
- L33 pad 1: Net-(L33-Pad1) -> VCC
- L33 pad 2: GND -> Net-(L33-Pad2)
- L33 pad 3: Net-(L32-Pad1) -> GND
- L33 pad 4: VCC -> Net-(L32-Pad2)
- L34 pad 1: Net-(L34-Pad1) -> VCC
- L34 pad 2: GND -> Net-(L34-Pad2)
- L34 pad 3: Net-(L33-Pad1) -> GND
- L34 pad 4: VCC -> Net-(L33-Pad2)
- L35 pad 1: Net-(L35-Pad1) -> VCC
- L35 pad 2: GND -> Net-(L35-Pad2)
- L35 pad 3: Net-(L34-Pad1) -> GND
- L35 pad 4: VCC -> Net-(L34-Pad2)
- L36 pad 1: Net-(L36-Pad1) -> VCC
- L36 pad 2: GND -> Net-(L36-Pad2)
- L36 pad 3: Net-(L35-Pad1) -> GND
- L36 pad 4: VCC -> Net-(L35-Pad2)
- L37 pad 1: Net-(L37-Pad1) -> VCC
- L37 pad 2: GND -> Net-(L37-Pad2)
- L37 pad 3: Net-(L36-Pad1) -> GND
- L37 pad 4: VCC -> Net-(L36-Pad2)
- L38 pad 1: Net-(L38-Pad1) -> VCC
- L38 pad 2: GND -> Net-(L38-Pad2)
- L38 pad 3: Net-(L37-Pad1) -> GND
- L38 pad 4: VCC -> Net-(L37-Pad2)
- L39 pad 1: Net-(L39-Pad1) -> VCC
- L39 pad 2: GND -> Net-(L39-Pad2)
- L39 pad 3: Net-(L38-Pad1) -> GND
- L39 pad 4: VCC -> Net-(L38-Pad2)
- L4 pad 1: Net-(L4-Pad1) -> VCC
- L4 pad 2: GND -> Net-(L4-Pad2)
- L4 pad 3: Net-(L3-Pad1) -> GND
- L4 pad 4: VCC -> Net-(L3-Pad2)
- L40 pad 1: Net-(L40-Pad1) -> VCC
- L40 pad 2: GND -> Net-(L40-Pad2)
- L40 pad 3: Net-(L39-Pad1) -> GND
- L40 pad 4: VCC -> Net-(L39-Pad2)
- L41 pad 1: Net-(L41-Pad1) -> VCC
- L41 pad 2: GND -> Net-(L41-Pad2)
- L41 pad 3: Net-(L40-Pad1) -> GND
- L41 pad 4: VCC -> Net-(L40-Pad2)
- L42 pad 1: Net-(L42-Pad1) -> VCC
- L42 pad 2: GND -> Net-(L42-Pad2)
- L42 pad 3: Net-(L41-Pad1) -> GND
- L42 pad 4: VCC -> Net-(L41-Pad2)
- L43 pad 1: Net-(L43-Pad1) -> VCC
- L43 pad 2: GND -> Net-(L43-Pad2)
- L43 pad 3: Net-(L42-Pad1) -> GND
- L43 pad 4: VCC -> Net-(L42-Pad2)
- L44 pad 1: Net-(L44-Pad1) -> VCC
- L44 pad 2: GND -> Net-(L44-Pad2)
- L44 pad 3: Net-(L43-Pad1) -> GND
- L44 pad 4: VCC -> Net-(L43-Pad2)
- L45 pad 1: Net-(L45-Pad1) -> VCC
- L45 pad 2: GND -> Net-(L45-Pad2)
- L45 pad 3: Net-(L44-Pad1) -> GND
- L45 pad 4: VCC -> Net-(L44-Pad2)
- L46 pad 1: Net-(L46-Pad1) -> VCC
- L46 pad 2: GND -> Net-(L46-Pad2)
- L46 pad 3: Net-(L45-Pad1) -> GND
- L46 pad 4: VCC -> Net-(L45-Pad2)
- L47 pad 1: Net-(L47-Pad1) -> VCC
- L47 pad 2: GND -> Net-(L47-Pad2)
- L47 pad 3: Net-(L46-Pad1) -> GND
- L47 pad 4: VCC -> Net-(L46-Pad2)
- L48 pad 1: Net-(L48-Pad1) -> VCC
- L48 pad 2: GND -> Net-(L48-Pad2)
- L48 pad 3: Net-(L47-Pad1) -> GND
- L48 pad 4: VCC -> Net-(L47-Pad2)
- L49 pad 1: Net-(L49-Pad1) -> VCC
- L49 pad 2: GND -> Net-(L49-Pad2)
- L49 pad 3: Net-(L48-Pad1) -> GND
- L49 pad 4: VCC -> Net-(L48-Pad2)
- L5 pad 1: Net-(L5-Pad1) -> VCC
- L5 pad 2: GND -> Net-(L5-Pad2)
- L5 pad 3: Net-(L4-Pad1) -> GND
- L5 pad 4: VCC -> Net-(L4-Pad2)
- L50 pad 1: Net-(L50-Pad1) -> VCC
- L50 pad 2: GND -> Net-(L50-Pad2)
- L50 pad 3: Net-(L49-Pad1) -> GND
- L50 pad 4: VCC -> Net-(L49-Pad2)
- L51 pad 1: Net-(L51-Pad1) -> VCC
- L51 pad 2: GND -> Net-(L51-Pad2)
- L51 pad 3: Net-(L50-Pad1) -> GND
- L51 pad 4: VCC -> Net-(L50-Pad2)
- L52 pad 1: Net-(L52-Pad1) -> VCC
- L52 pad 2: GND -> Net-(L52-Pad2)
- L52 pad 3: Net-(L51-Pad1) -> GND
- L52 pad 4: VCC -> Net-(L51-Pad2)
- L53 pad 1: Net-(L53-Pad1) -> VCC
- L53 pad 2: GND -> Net-(L53-Pad2)
- L53 pad 3: Net-(L52-Pad1) -> GND
- L53 pad 4: VCC -> Net-(L52-Pad2)
- L54 pad 1: Net-(J4-Pad2) -> VCC
- L54 pad 2: GND -> Net-(L54-Pad2)
- L54 pad 3: Net-(L53-Pad1) -> GND
- L54 pad 4: VCC -> Net-(L53-Pad2)
- L6 pad 1: Net-(L6-Pad1) -> VCC
- L6 pad 2: GND -> Net-(L6-Pad2)
- L6 pad 3: Net-(L5-Pad1) -> GND
- L6 pad 4: VCC -> Net-(L5-Pad2)
- L7 pad 1: Net-(L7-Pad1) -> VCC
- L7 pad 2: GND -> Net-(L7-Pad2)
- L7 pad 3: Net-(L6-Pad1) -> GND
- L7 pad 4: VCC -> Net-(L6-Pad2)
- L8 pad 1: Net-(L8-Pad1) -> VCC
- L8 pad 2: GND -> Net-(L8-Pad2)
- L8 pad 3: Net-(L7-Pad1) -> GND
- L8 pad 4: VCC -> Net-(L7-Pad2)
- L9 pad 1: Net-(L10-Pad3) -> VCC
- L9 pad 2: GND -> Net-(L10-Pad4)
- L9 pad 3: Net-(L8-Pad1) -> GND
- L9 pad 4: VCC -> Net-(L8-Pad2)
Routing:
- net GND: track 1235.6 -> 1646.9 mm, vias 38 -> 90
- net Net-(L27-Pad2): track 0.00 -> 115.4 mm, vias 0 -> 3
- net Net-(L55-Pad2): track 0.00 -> 93.6 mm, vias 0 -> 2
- net Net-(L4-Pad1): track 87.4 -> 0.00 mm, vias 4 -> 0
- net Net-(J4-Pad2): track 83.1 -> 0.00 mm, vias 4 -> 0
- net Net-(L51-Pad1): track 79.7 -> 0.00 mm
- net Net-(L4-Pad2): track 0.00 -> 77.8 mm, vias 0 -> 4
- net Net-(J2-Pad2): track 75.6 -> 0.00 mm, vias 2 -> 0
- net Net-(L24-Pad1): track 66.8 -> 0.00 mm, vias 2 -> 0
- net Net-(L52-Pad2): track 0.00 -> 62.8 mm, vias 0 -> 2
- net Net-(L24-Pad2): track 0.00 -> 62.6 mm, vias 0 -> 2
- net Net-(L53-Pad1): track 61.9 -> 0.00 mm, vias 4 -> 0
- net Net-(L32-Pad2): track 0.00 -> 60.2 mm, vias 0 -> 2
- net Net-(L54-Pad2): track 0.00 -> 58.7 mm, vias 0 -> 2
- net Net-(L31-Pad1): track 56.0 -> 0.00 mm, vias 2 -> 0
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- added copper zone on B.Cu, net GND
- added copper zone on F.Cu, net GND
Other:
- board size 288.1 x 124 mm -> 139.8 x 201 mm
- board text added: "@illness072"
- board text added: "Elephant42 [RC]"
- board text added: "HAPPY TYPING!!"
- board text added: "JLCJLCJLCJLC"
- board text added: "designed by"
- board text added: "inspired by claw44"

Commit message: small fix
Parts:
- RESET_SW1, RESET_SW2: footprint kbd:ResetSW -> phi-kbd-library:ResetSW-irreversible
- turned RESET_SW1 to 0 degrees
- turned RESET_SW2 to 0 degrees
Routing:
- net GND: vias 90 -> 88
- net (no net): vias 0 -> 2

Commit message: fix th
Parts:
- added J4: Conn_01x01, maou_kbd:M2hole, F.Cu at (21.7, 124.0)
- added J4: Conn_01x01, maou_kbd:M2hole, F.Cu at (34.7, 130.0)
- added J4: Conn_01x01, maou_kbd:M2hole, F.Cu at (142.4, 101.0)
- added J4: Conn_01x01, maou_kbd:M2hole, F.Cu at (129.4, 95.0)
- RESET_SW1, RESET_SW2: footprint phi-kbd-library:ResetSW-irreversible -> kbd:ResetSW_1side
- moved OL1 1.51 mm to (24.0, 145.0)
- moved OL2 1.20 mm to (132.7, 79.8)
- turned RESET_SW1 to 180 degrees
- turned RESET_SW2 to 180 degrees
Routing:
- net led_r: track 113.3 -> 126.9 mm
- net row7: track 150.5 -> 160.6 mm
- net col3: track 142.4 -> 149.7 mm
- net VCC: track 1240.1 -> 1246.6 mm, vias 39 -> 40
- net Net-(L54-Pad2): track 58.7 -> 52.4 mm
- net col9: track 186.0 -> 191.8 mm
- net col10: track 140.3 -> 145.1 mm
- net Net-(L4-Pad2): track 77.8 -> 80.7 mm
- net col4: track 116.9 -> 119.8 mm
- net col5: track 118.6 -> 121.5 mm
- net GND: track 1646.9 -> 1649.7 mm, vias 88 -> 92
- net led_l: track 121.1 -> 123.9 mm
- net sda_r: track 25.1 -> 27.3 mm
- net Net-(L31-Pad2): track 33.6 -> 31.7 mm
- net col11: track 127.2 -> 128.8 mm
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Other:
- outline, holes or cut-outs redrawn

Commit message: v1 pcb
Parts:
- added G***: LOGO, elephant42:icon_small, B.Cu at (82.5, 107.6)
- added G***: LOGO, elephant42:icon, F.Cu at (25.2, 115.2)
- added G***: LOGO, elephant42:icon, B.Cu at (137.6, 108.0)
Other:
- board text added: "elephant42 v1.0"
- board text added: "elephant42 v1.0 designed by illness072"
- board text removed: "Elephant42 [RC]"
- board text removed: "inspired by claw44"

Commit message: updat sch
Parts:
- D1, D10, D11, D12, D13, D14, D15, D16, D17, D18, D19, D2, D20, D21, D22, D23, D24, D25, D26, D27, D28, D29, D3, D30, D31, D32, D33, D34, D35, D36, D37, D38, D39, D4, D40, D41, D42, D5, D6, D7, D8, D9: footprint kbd:D3_SMD_v2 -> elephant42:D3_SMD_v2
- J1, J3: footprint kbd:MJ-4PP-9_1side -> elephant42:MJ-4PP-9_1side
- J4 (x4): footprint maou_kbd:M2hole -> elephant42:M2hole
- L1, L10, L11, L12, L13, L14, L15, L16, L17, L18, L19, L2, L20, L21, L29, L3, L30, L31, L32, L33, L34, L35, L36, L37, L38, L39, L4, L40, L41, L42, L43, L44, L45, L46, L47, L48, L49, L5, L6, L7, L8, L9: footprint maou_kbd:YS-SK6812MINI-E -> elephant42:YS-SK6812MINI-E
- L22, L23, L24, L25, L26, L27, L50, L51, L52, L53, L54, L55: footprint maou_kbd:YS-SK6812MINI-E-underglow -> elephant42:YS-SK6812MINI-E-underglow
- L28, L56: footprint kbd:StripLED_1side -> elephant42:StripLED_1side
- OL1, OL2: footprint kbd:OLED_1side -> elephant42:OLED_1side
- RESET_SW1, RESET_SW2: footprint kbd:ResetSW_1side -> elephant42:ResetSW_1side
- SW1, SW10, SW11, SW12, SW13, SW14, SW15, SW16, SW17, SW18, SW19, SW2, SW20, SW21, SW22, SW23, SW24, SW25, SW26, SW27, SW28, SW29, SW3, SW30, SW31, SW32, SW33, SW34, SW35, SW36, SW37, SW38, SW39, SW4, SW40, SW41, SW42, SW5, SW6, SW7, SW8, SW9: footprint kbd:CherryMX_Hotswap -> elephant42:CherryMX_Hotswap
- U1, U2: footprint kbd:ProMicro_v3 -> elephant42:ProMicro_v3
Connections:
- J1 pad A: (no net) -> Net-(J1-PadA)
- J3 pad A: (no net) -> Net-(J3-PadA)
- U1 pad 11: (no net) -> Net-(U1-Pad11)
- U1 pad 12: (no net) -> Net-(U1-Pad12)
- U1 pad 13: (no net) -> Net-(U1-Pad13)
- U1 pad 14: (no net) -> Net-(U1-Pad14)
- U1 pad 24: (no net) -> Net-(U1-Pad24)
- U2 pad 11: (no net) -> Net-(U2-Pad11)
- U2 pad 12: (no net) -> Net-(U2-Pad12)
- U2 pad 13: (no net) -> Net-(U2-Pad13)
- U2 pad 14: (no net) -> Net-(U2-Pad14)
- U2 pad 24: (no net) -> Net-(U2-Pad24)
